Commit message: Updated unstable urdf and sdf

File: urdf/husky.urdf (robot description, URDF)
Before this commit: robot husky, 32 links, 31 joints
Links:
- added link camera_link, mass 0.1; collision box size=.03 .03 .03; visual box size=.03 .03 .03
- added link camera_link_optical
Joints:
- added joint camera_joint: type fixed, parent base, child camera_link, origin xyz=0.225 0 0.075 rpy=0 0 0
- added joint camera_optical_joint: type fixed, parent camera_link, child camera_link_optical, origin xyz=0 0 0 rpy=-1.5707 0 -1.5707
- joint LF_ankle: axis 0.0 0.0 1.0 -> 
- joint LF_foot_fixed: origin xyz=0.0 0.0 0.0 rpy=0 0 0 -> xyz=0.01 0.0 0.0 rpy=0 0 0
- joint LH_foot_fixed: origin xyz=0.0 0.0 0.0 rpy=0 0 0 -> xyz=0.01 0.0 0.0 rpy=0 0 0
- joint RF_foot_fixed: origin xyz=0.0 0.0 0.0 rpy=0 0 0 -> xyz=0.01 0.0 0.0 rpy=0 0 0
- joint RH_ankle: axis 0.0 0.0 1.0 -> 
- joint RH_foot_fixed: origin xyz=0.0 0.0 0.0 rpy=0 0 0 -> xyz=0.01 0.0 0.0 rpy=0 0 0
- joint bl_control_rod: axis 0.0 0.0 1.0 -> 
- joint br_control_rod: axis 0.0 0.0 1.0 -> 
- joint fl_control_rod: axis 0.0 0.0 1.0 -> 
- joint fr_control_rod: axis 0.0 0.0 1.0 -> 
- joint hussain_imu_joint: origin xyz=0. 0. 0. rpy=0. 0. 0. -> xyz=0.01 0. 0. rpy=0. 0. 0.
- joint root_to_base_joint: origin xyz=0 0.0 0.0 rpy=0 0 0 -> xyz=0.01 0.0 0.0 rpy=0 0 0
- joint unitree_imu_joint: origin xyz=0. 0. 0. rpy=0. 0. 0. -> xyz=0.01 0. 0. rpy=0. 0. 0.
