Commit message: Upgraded with ros2_control

File: urdf/husky_description.urdf (robot description, URDF)
Before this commit: robot husky_description, 17 links, 16 joints
Links:
- removed link FL_Foot_Link
- removed link FL_Hip_Link
- removed link FL_Thigh_Link
- removed link FL_Tibia_Link
- removed link FR_Foot_Link
- removed link FR_Hip_Link
- removed link FR_Thigh_Link
- removed link FR_Tibia_Link
- removed link RL_Foot_Link
- removed link RL_Hip_Link
- removed link RL_Thigh_Link
- removed link RL_Tibia_Link
- removed link RR_Foot_Link
- removed link RR_Hip_Link
- removed link RR_Thigh_Link
- removed link RR_Tibia_Link
- removed link base_link
- added link LF_FOOT, mass 0.06; collision sphere radius=${foot_sphere_radius}
- added link LF_calf, mass 0.05; collision cylinder length=${tibia_length} radius=${tibia_radius}; visual mesh filename=package://husky_description/meshes/fr_tibia.STL scale=1 1 1
- added link LF_fut, mass 0.05; collision cylinder length=${foot_length} radius=${foot_radius}; visual mesh filename=package://husky_description/meshes/fr_foot.STL scale=1 1 1
- added link LF_hip, mass 0.02; collision cylinder length=${hip_length} radius=${hip_radius}; visual mesh filename=package://husky_description/meshes/bl_hip.STL scale=1 1 1
- added link LF_thigh, mass 0.2; collision cylinder length=${femur_length} radius=${femur_radius}; collision cylinder length=${femur_n1_length} radius=${femur_n1_radius}
- added link LH_FOOT, mass 0.06; collision sphere radius=${foot_sphere_radius}
- added link LH_calf, mass 0.05; collision cylinder length=${tibia_length} radius=${tibia_radius}; visual mesh filename=package://husky_description/meshes/fr_tibia.STL scale=1 1 1
- added link LH_fut, mass 0.05; collision cylinder length=${foot_length} radius=${foot_radius}; visual mesh filename=package://husky_description/meshes/fr_foot.STL scale=1 1 1
- added link LH_hip, mass 0.02; collision cylinder length=${hip_length} radius=${hip_radius}; visual mesh filename=package://husky_description/meshes/bl_hip.STL scale=1 1 1
- added link LH_thigh, mass 0.2; collision cylinder length=${femur_length} radius=${femur_radius}; collision cylinder length=${femur_n1_length} radius=${femur_n1_radius}
- added link RF_FOOT, mass 0.06; collision sphere radius=${foot_sphere_radius}
- added link RF_calf, mass 0.05; collision cylinder length=${tibia_length} radius=${tibia_radius}; visual mesh filename=package://husky_description/meshes/fr_tibia.STL scale=1 1 1
- added link RF_fut, mass 0.05; collision cylinder length=${foot_length} radius=${foot_radius}; visual mesh filename=package://husky_description/meshes/fr_foot.STL scale=1 1 1
- added link RF_hip, mass 0.02; collision cylinder length=${hip_length} radius=${hip_radius}; visual mesh filename=package://husky_description/meshes/fr_hip.STL scale=1 1 1
- added link RF_thigh, mass 0.2; collision cylinder length=${femur_length} radius=${femur_radius}; collision cylinder length=${femur_n1_length} radius=${femur_n1_radius}
- added link RH_FOOT, mass 0.06; collision sphere radius=${foot_sphere_radius}
- added link RH_calf, mass 0.05; collision cylinder length=${tibia_length} radius=${tibia_radius}; visual mesh filename=package://husky_description/meshes/fr_tibia.STL scale=1 1 1
- added link RH_fut, mass 0.05; collision cylinder length=${foot_length} radius=${foot_radius}; visual mesh filename=package://husky_description/meshes/fr_foot.STL scale=1 1 1
- added link RH_hip, mass 0.02; collision cylinder length=${hip_length} radius=${hip_radius}; visual mesh filename=package://husky_description/meshes/fr_hip.STL scale=1 1 1
- added link RH_thigh, mass 0.2; collision cylinder length=${femur_length} radius=${femur_radius}; collision cylinder length=${femur_n1_length} radius=${femur_n1_radius}
- added link base, mass 3.1895; collision box size=0.3 0.1 0.12; collision box size=0.4 0.16 0.32
- added link bl_fibula, mass 0.020; collision cylinder length=${fibula_length} radius=${fibula_radius}; visual mesh filename=package://husky_description/meshes/fr_fibula.STL scale=1 1 1
- added link br_fibula, mass 0.020; collision cylinder length=${fibula_length} radius=${fibula_radius}; visual mesh filename=package://husky_description/meshes/fr_fibula.STL scale=1 1 1
- added link fl_fibula, mass 0.020; collision cylinder length=${fibula_length} radius=${fibula_radius}; visual mesh filename=package://husky_description/meshes/fr_fibula.STL scale=1 1 1
- added link fr_fibula, mass 0.020; collision cylinder length=${fibula_length} radius=${fibula_radius}; visual mesh filename=package://husky_description/meshes/fr_fibula.STL scale=1 1 1
- added link root
Joints:
- removed joint FL_H_F
- removed joint FL_H_S
- removed joint FL_T_A
- removed joint FL_T_K
- removed joint FR_H_F
- removed joint FR_H_S
- removed joint FR_T_A
- removed joint FR_T_K
- removed joint RL_H_F
- removed joint RL_H_S
- removed joint RL_T_A
- removed joint RL_T_K
- removed joint RR_H_F
- removed joint RR_H_S
- removed joint RR_T_A
- removed joint RR_T_K
- added joint LF_HAA: type revolute, parent base, child LF_hip, origin xyz=0.2087 0.045 0.0001 rpy=-1.5708 ${l_hip_frontal_ipos} -1.5708, axis 0.0 0.0 1.0, limit lower=${l_hip_frontal_lowlim} upper=${l_hip_frontal_uplim} effort=${efflim} velocity=8.7267
- added joint LF_HFE: type revolute, parent LF_hip, child LF_thigh, origin xyz=0.1031 0.0 0.0 rpy=-1.5708 ${fl_hip_sagittal_ipos} -1.5708, axis 0.0 0.0 ${l_axis}, limit lower=${fl_hip_sagittal_lowlim} upper=${fl_hip_sagittal_uplim} effort=${efflim} velocity=8.7267
- added joint LF_KFE: type revolute, parent LF_thigh, child LF_calf, origin xyz=0.18 0.0 -0.0431 rpy=0 0 ${l_knee_ipos}, axis 0.0 0.0 ${l_axis}, limit lower=${l_knee_lowlim} upper=${l_knee_uplim} effort=${efflim} velocity=8.7267
- added joint LF_ankle: type revolute, parent LF_calf, child LF_fut, origin xyz=0.333 0.0 0.0 rpy=0 0 ${r_knee_ipos}, axis 0.0 0.0 1.0, limit lower=${l_ankle_lowlim} upper=${l_ankle_uplim} effort=${efflim} velocity=8.7267, mimic joint=LF_KFE multiplier=-1
- added joint LF_foot_fixed: type fixed, parent LF_fut, child LF_FOOT, origin xyz=0.0 0.0 0.0 rpy=0 0 0
- added joint LH_HAA: type revolute, parent base, child LH_hip, origin xyz=-0.1862 0.045 0.0002 rpy=-1.5708 ${l_hip_frontal_ipos} -1.5708, axis 0.0 0.0 1.0, limit lower=${l_hip_frontal_lowlim} upper=${l_hip_frontal_uplim} effort=${efflim} velocity=8.7267
- added joint LH_HFE: type revolute, parent LH_hip, child LH_thigh, origin xyz=0.1031 0.0 0.0 rpy=-1.5708 ${bl_hip_sagittal_ipos} -1.5708, axis 0.0 0.0 ${l_axis}, limit lower=${bl_hip_sagittal_lowlim} upper=${bl_hip_sagittal_uplim} effort=${efflim} velocity=8.7267
- added joint LH_KFE: type revolute, parent LH_thigh, child LH_calf, origin xyz=0.18 0.0 -0.0431 rpy=0 0 ${l_knee_ipos}, axis 0.0 0.0 ${l_axis}, limit lower=${l_knee_lowlim} upper=${l_knee_uplim} effort=${efflim} velocity=8.7267
- added joint LH_ankle: type revolute, parent LH_calf, child LH_fut, origin xyz=0.333 0.0 0.0 rpy=0 0 ${r_knee_ipos}, axis 0.0 0.0 1.0, limit lower=${l_ankle_lowlim} upper=${l_ankle_uplim} effort=${efflim} velocity=8.7267, mimic joint=LH_KFE multiplier=-1
- added joint LH_foot_fixed: type fixed, parent LH_fut, child LH_FOOT, origin xyz=0.0 0.0 0.0 rpy=0 0 0
- added joint RF_HAA: type revolute, parent base, child RF_hip, origin xyz=0.2087 -0.045 0.0001 rpy=-1.5708 ${r_hip_frontal_ipos} -1.5708, axis 0.0 0.0 1.0, limit lower=${r_hip_frontal_lowlim} upper=${r_hip_frontal_uplim} effort=${efflim} velocity=8.7267
- added joint RF_HFE: type revolute, parent RF_hip, child RF_thigh, origin xyz=0.1031 0.0 0.0 rpy=-1.5708 ${fr_hip_sagittal_ipos} -1.5708, axis 0.0 0.0 ${r_axis}, limit lower=${fr_hip_sagittal_lowlim} upper=${fr_hip_sagittal_uplim} effort=${efflim} velocity=8.7267
- added joint RF_KFE: type revolute, parent RF_thigh, child RF_calf, origin xyz=0.18 0.0 -0.0431 rpy=0 0 ${r_knee_ipos}, axis 0.0 0.0 ${r_axis}, limit lower=${r_knee_lowlim} upper=${r_knee_uplim} effort=${efflim} velocity=8.7267
- added joint RF_ankle: type revolute, parent RF_calf, child RF_fut, origin xyz=0.333 0.0 0.0 rpy=0 0 ${l_knee_ipos}, axis 0.0 0.0 1.0, limit lower=${r_ankle_lowlim} upper=${r_ankle_uplim} effort=${efflim} velocity=8.7267, mimic joint=RF_KFE multiplier=-1
- added joint RF_foot_fixed: type fixed, parent RF_fut, child RF_FOOT, origin xyz=0.0 0.0 0.0 rpy=0 0 0
- added joint RH_HAA: type revolute, parent base, child RH_hip, origin xyz=-0.1862 -0.045 0.0002 rpy=-1.5708 ${r_hip_frontal_ipos} -1.5708, axis 0.0 0.0 1.0, limit lower=${r_hip_frontal_lowlim} upper=${r_hip_frontal_uplim} effort=${efflim} velocity=8.7267
- added joint RH_HFE: type revolute, parent RH_hip, child RH_thigh, origin xyz=0.1031 0.0 0.0 rpy=-1.5708 ${br_hip_sagittal_ipos} -1.5708, axis 0.0 0.0 ${r_axis}, limit lower=${br_hip_sagittal_lowlim} upper=${br_hip_sagittal_uplim} effort=${efflim} velocity=8.7267
- added joint RH_KFE: type revolute, parent RH_thigh, child RH_calf, origin xyz=0.18 0.0 -0.0431 rpy=0 0 ${r_knee_ipos}, axis 0.0 0.0 ${r_axis}, limit lower=${r_knee_lowlim} upper=${r_knee_uplim} effort=${efflim} velocity=8.7267
- added joint RH_ankle: type revolute, parent RH_calf, child RH_fut, origin xyz=0.333 0.0 0.0 rpy=0 0 ${l_knee_ipos}, axis 0.0 0.0 1.0, limit lower=${r_ankle_lowlim} upper=${r_ankle_uplim} effort=${efflim} velocity=8.7267, mimic joint=RH_KFE multiplier=-1
- added joint RH_foot_fixed: type fixed, parent RH_fut, child RH_FOOT, origin xyz=0.0 0.0 0.0 rpy=0 0 0
- added joint bl_control_rod: type revolute, parent LH_thigh, child bl_fibula, origin xyz=0.12 0.0 -0.0431 rpy=0 0.0 ${l_knee_ipos}, axis 0.0 0.0 1.0, limit lower=${l_knee_lowlim} upper=${l_knee_uplim} effort=${efflim} velocity=8.7267, mimic joint=LH_KFE multiplier=1
- added joint br_control_rod: type revolute, parent RH_thigh, child br_fibula, origin xyz=0.12 0.0 -0.0431 rpy=0 0.0 ${r_knee_ipos}, axis 0.0 0.0 1.0, limit lower=${r_knee_lowlim} upper=${r_knee_uplim} effort=${efflim} velocity=8.7267, mimic joint=RH_KFE multiplier=1
- added joint fl_control_rod: type revolute, parent LF_thigh, child fl_fibula, origin xyz=0.12 0.0 -0.0431 rpy=0 0.0 ${l_knee_ipos}, axis 0.0 0.0 1.0, limit lower=${l_knee_lowlim} upper=${l_knee_uplim} effort=${efflim} velocity=8.7267, mimic joint=LF_KFE multiplier=1
- added joint fr_control_rod: type revolute, parent RF_thigh, child fr_fibula, origin xyz=0.12 0.0 -0.0431 rpy=0 0.0 ${r_knee_ipos}, axis 0.0 0.0 1.0, limit lower=${r_knee_lowlim} upper=${r_knee_uplim} effort=${efflim} velocity=8.7267, mimic joint=RF_KFE multiplier=1
- added joint root_to_base_joint: type fixed, parent root, child base, origin xyz=0 0.0 0.0 rpy=0 0 0

Commit message: Modified and fixed controller issues

File: urdf/husky_description.urdf (robot description, URDF)
Before this commit: robot husky, 26 links, 25 joints
Links:
- link LF_FOOT: geometry collision sphere radius=0.02
- link LF_calf: geometry collision cylinder length=0.32 radius=0.01; visual mesh filename=package://husky_description/meshes/fr_tibia.STL scale=1 1 1
- link LF_fut: geometry collision cylinder length=0.16 radius=0.01; visual mesh filename=package://husky_description/meshes/fr_foot.STL scale=1 1 1
- link LF_hip: geometry collision cylinder length=0.08 radius=0.03; visual mesh filename=package://husky_description/meshes/bl_hip.STL scale=1 1 1
- link LF_thigh: geometry collision cylinder length=0.05 radius=0.03; collision cylinder length=0.06 radius=0.03
- link LH_FOOT: geometry collision sphere radius=0.02
- link LH_calf: geometry collision cylinder length=0.32 radius=0.01; visual mesh filename=package://husky_description/meshes/fr_tibia.STL scale=1 1 1
- link LH_fut: geometry collision cylinder length=0.16 radius=0.01; visual mesh filename=package://husky_description/meshes/fr_foot.STL scale=1 1 1
- link LH_hip: geometry collision cylinder length=0.08 radius=0.03; visual mesh filename=package://husky_description/meshes/bl_hip.STL scale=1 1 1
- link LH_thigh: geometry collision cylinder length=0.05 radius=0.03; collision cylinder length=0.06 radius=0.03
- link RF_FOOT: geometry collision sphere radius=0.02
- link RF_calf: geometry collision cylinder length=0.32 radius=0.01; visual mesh filename=package://husky_description/meshes/fr_tibia.STL scale=1 1 1
- link RF_fut: geometry collision cylinder length=0.16 radius=0.01; visual mesh filename=package://husky_description/meshes/fr_foot.STL scale=1 1 1
- link RF_hip: geometry collision cylinder length=0.08 radius=0.03; visual mesh filename=package://husky_description/meshes/fr_hip.STL scale=1 1 1
- link RF_thigh: geometry collision cylinder length=0.05 radius=0.03; collision cylinder length=0.06 radius=0.03
- link RH_FOOT: geometry collision sphere radius=0.02
- link RH_calf: geometry collision cylinder length=0.32 radius=0.01; visual mesh filename=package://husky_description/meshes/fr_tibia.STL scale=1 1 1
- link RH_fut: geometry collision cylinder length=0.16 radius=0.01; visual mesh filename=package://husky_description/meshes/fr_foot.STL scale=1 1 1
- link RH_hip: geometry collision cylinder length=0.08 radius=0.03; visual mesh filename=package://husky_description/meshes/fr_hip.STL scale=1 1 1
- link RH_thigh: geometry collision cylinder length=0.05 radius=0.03; collision cylinder length=0.06 radius=0.03
- link bl_fibula: geometry collision cylinder length=0.24 radius=0.01; visual mesh filename=package://husky_description/meshes/fr_fibula.STL scale=1 1 1
- link br_fibula: geometry collision cylinder length=0.24 radius=0.01; visual mesh filename=package://husky_description/meshes/fr_fibula.STL scale=1 1 1
- link fl_fibula: geometry collision cylinder length=0.24 radius=0.01; visual mesh filename=package://husky_description/meshes/fr_fibula.STL scale=1 1 1
- link fr_fibula: geometry collision cylinder length=0.24 radius=0.01; visual mesh filename=package://husky_description/meshes/fr_fibula.STL scale=1 1 1
Joints:
- joint LF_HAA: limit lower=${l_hip_frontal_lowlim} upper=${l_hip_frontal_uplim} effort=${efflim} velocity=8.7267 -> lower=0.08726646259971647 upper=0.4363323129985824 effort=33.5 velocity=8.7267; origin xyz=0.2087 0.045 0.0001 rpy=-1.5708 ${l_hip_frontal_ipos} -1.5708 -> xyz=0.2087 0.045 0.0001 rpy=-1.5708 -3.141592653589793 -1.5708
- joint LF_HFE: axis 0.0 0.0 ${l_axis} -> 0.0 0.0 1; limit lower=${fl_hip_sagittal_lowlim} upper=${fl_hip_sagittal_uplim} effort=${efflim} velocity=8.7267 -> lower=0.4363323129985824 upper=1.1344640137963142 effort=33.5 velocity=8.7267; origin xyz=0.1031 0.0 0.0 rpy=-1.5708 ${fl_hip_sagittal_ipos} -1.5708 -> xyz=0.1031 0.0 0.0 rpy=-1.5708 4.71238898038469 -1.5708
- joint LF_KFE: axis 0.0 0.0 ${l_axis} -> 0.0 0.0 1; limit lower=${l_knee_lowlim} upper=${l_knee_uplim} effort=${efflim} velocity=8.7267 -> lower=-1.8675022996339325 upper=-0.7330382858376184 effort=33.5 velocity=8.7267; origin xyz=0.18 0.0 -0.0431 rpy=0 0 ${l_knee_ipos} -> xyz=0.18 0.0 -0.0431 rpy=0 0 3.141592653589793
- joint LF_ankle: limit lower=${l_ankle_lowlim} upper=${l_ankle_uplim} effort=${efflim} velocity=8.7267 -> lower=-1.5707963267948966 upper=1.5707963267948966 effort=33.5 velocity=8.7267; origin xyz=0.333 0.0 0.0 rpy=0 0 ${r_knee_ipos} -> xyz=0.333 0.0 0.0 rpy=0 0 -3.141592653589793
- joint LH_HAA: limit lower=${l_hip_frontal_lowlim} upper=${l_hip_frontal_uplim} effort=${efflim} velocity=8.7267 -> lower=0.08726646259971647 upper=0.4363323129985824 effort=33.5 velocity=8.7267; origin xyz=-0.1862 0.045 0.0002 rpy=-1.5708 ${l_hip_frontal_ipos} -1.5708 -> xyz=-0.1862 0.045 0.0002 rpy=-1.5708 -3.141592653589793 -1.5708
- joint LH_HFE: axis 0.0 0.0 ${l_axis} -> 0.0 0.0 1; limit lower=${bl_hip_sagittal_lowlim} upper=${bl_hip_sagittal_uplim} effort=${efflim} velocity=8.7267 -> lower=0.4363323129985824 upper=1.1344640137963142 effort=33.5 velocity=8.7267; origin xyz=0.1031 0.0 0.0 rpy=-1.5708 ${bl_hip_sagittal_ipos} -1.5708 -> xyz=0.1031 0.0 0.0 rpy=-1.5708 4.71238898038469 -1.5708
- joint LH_KFE: axis 0.0 0.0 ${l_axis} -> 0.0 0.0 1; limit lower=${l_knee_lowlim} upper=${l_knee_uplim} effort=${efflim} velocity=8.7267 -> lower=-1.8675022996339325 upper=-0.7330382858376184 effort=33.5 velocity=8.7267; origin xyz=0.18 0.0 -0.0431 rpy=0 0 ${l_knee_ipos} -> xyz=0.18 0.0 -0.0431 rpy=0 0 3.141592653589793
- joint LH_ankle: limit lower=${l_ankle_lowlim} upper=${l_ankle_uplim} effort=${efflim} velocity=8.7267 -> lower=-1.5707963267948966 upper=1.5707963267948966 effort=33.5 velocity=8.7267; origin xyz=0.333 0.0 0.0 rpy=0 0 ${r_knee_ipos} -> xyz=0.333 0.0 0.0 rpy=0 0 -3.141592653589793
- joint RF_HAA: limit lower=${r_hip_frontal_lowlim} upper=${r_hip_frontal_uplim} effort=${efflim} velocity=8.7267 -> lower=-0.4363323129985824 upper=-0.08726646259971647 effort=33.5 velocity=8.7267; origin xyz=0.2087 -0.045 0.0001 rpy=-1.5708 ${r_hip_frontal_ipos} -1.5708 -> xyz=0.2087 -0.045 0.0001 rpy=-1.5708 0.0 -1.5708
- joint RF_HFE: axis 0.0 0.0 ${r_axis} -> 0.0 0.0 1; limit lower=${fr_hip_sagittal_lowlim} upper=${fr_hip_sagittal_uplim} effort=${efflim} velocity=8.7267 -> lower=-1.1344640137963142 upper=-0.4363323129985824 effort=33.5 velocity=8.7267; origin xyz=0.1031 0.0 0.0 rpy=-1.5708 ${fr_hip_sagittal_ipos} -1.5708 -> xyz=0.1031 0.0 0.0 rpy=-1.5708 -1.5707963267948966 -1.5708
- joint RF_KFE: axis 0.0 0.0 ${r_axis} -> 0.0 0.0 1; limit lower=${r_knee_lowlim} upper=${r_knee_uplim} effort=${efflim} velocity=8.7267 -> lower=0.7330382858376184 upper=1.8675022996339325 effort=33.5 velocity=8.7267; origin xyz=0.18 0.0 -0.0431 rpy=0 0 ${r_knee_ipos} -> xyz=0.18 0.0 -0.0431 rpy=0 0 -3.141592653589793
- joint RF_ankle: limit lower=${r_ankle_lowlim} upper=${r_ankle_uplim} effort=${efflim} velocity=8.7267 -> lower=-1.5707963267948966 upper=1.5707963267948966 effort=33.5 velocity=8.7267; origin xyz=0.333 0.0 0.0 rpy=0 0 ${l_knee_ipos} -> xyz=0.333 0.0 0.0 rpy=0 0 3.141592653589793
- joint RH_HAA: limit lower=${r_hip_frontal_lowlim} upper=${r_hip_frontal_uplim} effort=${efflim} velocity=8.7267 -> lower=-0.4363323129985824 upper=-0.08726646259971647 effort=33.5 velocity=8.7267; origin xyz=-0.1862 -0.045 0.0002 rpy=-1.5708 ${r_hip_frontal_ipos} -1.5708 -> xyz=-0.1862 -0.045 0.0002 rpy=-1.5708 0.0 -1.5708
- joint RH_HFE: axis 0.0 0.0 ${r_axis} -> 0.0 0.0 1; limit lower=${br_hip_sagittal_lowlim} upper=${br_hip_sagittal_uplim} effort=${efflim} velocity=8.7267 -> lower=-1.1344640137963142 upper=-0.4363323129985824 effort=33.5 velocity=8.7267; origin xyz=0.1031 0.0 0.0 rpy=-1.5708 ${br_hip_sagittal_ipos} -1.5708 -> xyz=0.1031 0.0 0.0 rpy=-1.5708 -1.5707963267948966 -1.5708
- joint RH_KFE: axis 0.0 0.0 ${r_axis} -> 0.0 0.0 1; limit lower=${r_knee_lowlim} upper=${r_knee_uplim} effort=${efflim} velocity=8.7267 -> lower=0.7330382858376184 upper=1.8675022996339325 effort=33.5 velocity=8.7267; origin xyz=0.18 0.0 -0.0431 rpy=0 0 ${r_knee_ipos} -> xyz=0.18 0.0 -0.0431 rpy=0 0 -3.141592653589793
- joint RH_ankle: limit lower=${r_ankle_lowlim} upper=${r_ankle_uplim} effort=${efflim} velocity=8.7267 -> lower=-1.5707963267948966 upper=1.5707963267948966 effort=33.5 velocity=8.7267; origin xyz=0.333 0.0 0.0 rpy=0 0 ${l_knee_ipos} -> xyz=0.333 0.0 0.0 rpy=0 0 3.141592653589793
- joint bl_control_rod: limit lower=${l_knee_lowlim} upper=${l_knee_uplim} effort=${efflim} velocity=8.7267 -> lower=-1.8675022996339325 upper=-0.7330382858376184 effort=33.5 velocity=8.7267; origin xyz=0.12 0.0 -0.0431 rpy=0 0.0 ${l_knee_ipos} -> xyz=0.12 0.0 -0.0431 rpy=0 0.0 3.141592653589793
- joint br_control_rod: limit lower=${r_knee_lowlim} upper=${r_knee_uplim} effort=${efflim} velocity=8.7267 -> lower=0.7330382858376184 upper=1.8675022996339325 effort=33.5 velocity=8.7267; origin xyz=0.12 0.0 -0.0431 rpy=0 0.0 ${r_knee_ipos} -> xyz=0.12 0.0 -0.0431 rpy=0 0.0 -3.141592653589793
- joint fl_control_rod: limit lower=${l_knee_lowlim} upper=${l_knee_uplim} effort=${efflim} velocity=8.7267 -> lower=-1.8675022996339325 upper=-0.7330382858376184 effort=33.5 velocity=8.7267; origin xyz=0.12 0.0 -0.0431 rpy=0 0.0 ${l_knee_ipos} -> xyz=0.12 0.0 -0.0431 rpy=0 0.0 3.141592653589793
- joint fr_control_rod: limit lower=${r_knee_lowlim} upper=${r_knee_uplim} effort=${efflim} velocity=8.7267 -> lower=0.7330382858376184 upper=1.8675022996339325 effort=33.5 velocity=8.7267; origin xyz=0.12 0.0 -0.0431 rpy=0 0.0 ${r_knee_ipos} -> xyz=0.12 0.0 -0.0431 rpy=0 0.0 -3.141592653589793
