Commit message: Fixed JointTrajectoryController

File: urdf/husky_description.urdf (robot description, URDF)
Before this commit: robot husky, 26 links, 25 joints
Links:
- added link camera_link, mass 0.1; collision box size=.03 .03 .03; visual box size=.03 .03 .03
- added link camera_link_optical
- added link imu_link
- link LF_FOOT: geometry collision sphere radius=0.02; visual sphere radius=0.02
- link LH_FOOT: geometry collision sphere radius=0.02; visual sphere radius=0.02
- link RF_FOOT: geometry collision sphere radius=0.02; visual sphere radius=0.02
- link RH_FOOT: geometry collision sphere radius=0.02; visual sphere radius=0.02
Joints:
- added joint camera_joint: type fixed, parent base, child camera_link, origin xyz=0.225 0 0.075 rpy=0 0 0, axis 0 1 0
- added joint camera_optical_joint: type fixed, parent camera_link, child camera_link_optical, origin xyz=0 0 0 rpy=-1.5707 0 -1.5707
- added joint imu_joint: type fixed, parent base, child imu_link, origin xyz=0 0 0 rpy=0 0 0
- joint LF_HAA: limit lower=0.08726646259971647 upper=0.4363323129985824 effort=33.5 velocity=8.7267 -> lower=0.08726646259971647 upper=0.4363323129985824 effort=23.5 velocity=8.7267
- joint LF_HFE: limit lower=0.4363323129985824 upper=1.1344640137963142 effort=33.5 velocity=8.7267 -> lower=0.4363323129985824 upper=1.1344640137963142 effort=23.5 velocity=8.7267
- joint LF_KFE: limit lower=-1.8675022996339325 upper=-0.7330382858376184 effort=33.5 velocity=8.7267 -> lower=-1.8675022996339325 upper=-0.7330382858376184 effort=23.5 velocity=8.7267
- joint LF_ankle: limit lower=-1.5707963267948966 upper=1.5707963267948966 effort=33.5 velocity=8.7267 -> lower=-1.5707963267948966 upper=1.5707963267948966 effort=23.5 velocity=8.7267
- joint LH_HAA: limit lower=0.08726646259971647 upper=0.4363323129985824 effort=33.5 velocity=8.7267 -> lower=0.08726646259971647 upper=0.4363323129985824 effort=23.5 velocity=8.7267
- joint LH_HFE: limit lower=0.4363323129985824 upper=1.1344640137963142 effort=33.5 velocity=8.7267 -> lower=0.4363323129985824 upper=1.1344640137963142 effort=23.5 velocity=8.7267
- joint LH_KFE: limit lower=-1.8675022996339325 upper=-0.7330382858376184 effort=33.5 velocity=8.7267 -> lower=-1.8675022996339325 upper=-0.7330382858376184 effort=23.5 velocity=8.7267
- joint LH_ankle: limit lower=-1.5707963267948966 upper=1.5707963267948966 effort=33.5 velocity=8.7267 -> lower=-1.5707963267948966 upper=1.5707963267948966 effort=23.5 velocity=8.7267
- joint RF_HAA: limit lower=-0.4363323129985824 upper=-0.08726646259971647 effort=33.5 velocity=8.7267 -> lower=-0.4363323129985824 upper=-0.08726646259971647 effort=23.5 velocity=8.7267
- joint RF_HFE: limit lower=-1.1344640137963142 upper=-0.4363323129985824 effort=33.5 velocity=8.7267 -> lower=-1.1344640137963142 upper=-0.4363323129985824 effort=23.5 velocity=8.7267
- joint RF_KFE: limit lower=0.7330382858376184 upper=1.8675022996339325 effort=33.5 velocity=8.7267 -> lower=0.7330382858376184 upper=1.8675022996339325 effort=23.5 velocity=8.7267
- joint RF_ankle: limit lower=-1.5707963267948966 upper=1.5707963267948966 effort=33.5 velocity=8.7267 -> lower=-1.5707963267948966 upper=1.5707963267948966 effort=23.5 velocity=8.7267
- joint RH_HAA: limit lower=-0.4363323129985824 upper=-0.08726646259971647 effort=33.5 velocity=8.7267 -> lower=-0.4363323129985824 upper=-0.08726646259971647 effort=23.5 velocity=8.7267
- joint RH_HFE: limit lower=-1.1344640137963142 upper=-0.4363323129985824 effort=33.5 velocity=8.7267 -> lower=-1.1344640137963142 upper=-0.4363323129985824 effort=23.5 velocity=8.7267
- joint RH_KFE: limit lower=0.7330382858376184 upper=1.8675022996339325 effort=33.5 velocity=8.7267 -> lower=0.7330382858376184 upper=1.8675022996339325 effort=23.5 velocity=8.7267
- joint RH_ankle: limit lower=-1.5707963267948966 upper=1.5707963267948966 effort=33.5 velocity=8.7267 -> lower=-1.5707963267948966 upper=1.5707963267948966 effort=23.5 velocity=8.7267
- joint bl_control_rod: limit lower=-1.8675022996339325 upper=-0.7330382858376184 effort=33.5 velocity=8.7267 -> lower=-1.8675022996339325 upper=-0.7330382858376184 effort=23.5 velocity=8.7267
- joint br_control_rod: limit lower=0.7330382858376184 upper=1.8675022996339325 effort=33.5 velocity=8.7267 -> lower=0.7330382858376184 upper=1.8675022996339325 effort=23.5 velocity=8.7267
- joint fl_control_rod: limit lower=-1.8675022996339325 upper=-0.7330382858376184 effort=33.5 velocity=8.7267 -> lower=-1.8675022996339325 upper=-0.7330382858376184 effort=23.5 velocity=8.7267
- joint fr_control_rod: limit lower=0.7330382858376184 upper=1.8675022996339325 effort=33.5 velocity=8.7267 -> lower=0.7330382858376184 upper=1.8675022996339325 effort=23.5 velocity=8.7267

File: urdf/husky_description.xacro (robot description, xacro)
@@ -809,5 +809,10 @@
       <always_on>true</always_on>
       <update_rate>100.0</update_rate>
-      <topic>/rf_foot/contacts</topic>
+      <plugin name="gazebo_ros_contact_rf" filename="gz_ros2_contact_sensor_system">
+        <ros>
+          <namespace>/rf_foot</namespace>
+          <remapping>~/contacts:=contacts</remapping>
+        </ros>
+      </plugin>
     </sensor>
   </link>
@@ -832,5 +837,10 @@
       <always_on>true</always_on>
       <update_rate>100.0</update_rate>
-      <topic>/lf_foot/contacts</topic>
+      <plugin name="gazebo_ros_contact_lf" filename="gz_ros2_contact_sensor_system">
+        <ros>
+          <namespace>/lf_foot</namespace>
+          <remapping>~/contacts:=contacts</remapping>
+        </ros>
+      </plugin>
     </sensor>
   </link>
@@ -855,5 +865,10 @@
       <always_on>true</always_on>
       <update_rate>100.0</update_rate>
-      <topic>/lh_foot/contacts</topic>
+      <plugin name="gazebo_ros_contact_lh" filename="gz_ros2_contact_sensor_system">
+        <ros>
+          <namespace>/lh_foot</namespace>
+          <remapping>~/contacts:=contacts</remapping>
+        </ros>
+      </plugin>
     </sensor>
   </link>
@@ -878,5 +893,10 @@
       <always_on>true</always_on>
       <update_rate>100.0</update_rate>
-      <topic>/rh_foot/contacts</topic>
+      <plugin name="gazebo_ros_contact_rh" filename="gz_ros2_contact_sensor_system">
+        <ros>
+          <namespace>/rh_foot</namespace>
+          <remapping>~/contacts:=contacts</remapping>
+        </ros>
+      </plugin>
     </sensor>
   </link>
@@ -1170,112 +1190,113 @@
   </transmission>
   <ros2_control name="GazeboSystem" type="system">
-      <hardware>
-        <plugin>gz_ros2_control/GazeboSimSystem</plugin>
-        <!-- 🔧 Force joint interfaces to be POSITION -->
-        <param name="command_interface">position</param>
-      </hardware>
-      <!-- 12 Actuated Joints (Effort-Controlled) -->
-      <joint name="RF_HAA">
-          <command_interface name="effort"/>
-          <state_interface name="position"/>
-          <state_interface name="velocity"/>
-          <param name="command_interface">position</param>
-      </joint>
-      <joint name="RF_HFE">
-          <command_interface name="effort"/>
-          <state_interface name="position"/>
-          <state_interface name="velocity"/>
-          <param name="command_interface">position</param>
-      </joint>
-      <joint name="RF_KFE">
-          <command_interface name="effort"/>
-          <state_interface name="position"/>
-          <state_interface name="velocity"/>
-          <param name="command_interface">position</param>
-      </joint>
-      <joint name="LF_HAA">
-          <command_interface name="effort"/>
-          <state_interface name="position"/>
-          <state_interface name="velocity"/>
-          <param name="command_interface">position</param>
-      </joint>
-      <joint name="LF_HFE">
-          <command_interface name="effort"/>
-          <state_interface name="position"/>
-          <state_interface name="velocity"/>
-          <param name="command_interface">position</param>
-      </joint>
-      <joint name="LF_KFE">
-          <command_interface name="effort"/>
-          <state_interface name="position"/>
-          <state_interface name="velocity"/>
-          <param name="command_interface">position</param>
-      </joint>
-      <joint name="RH_HAA">
-          <command_interface name="effort"/>
-          <state_interface name="position"/>
-          <state_interface name="velocity"/>
-          <param name="command_interface">position</param>
-      </joint>
-      <joint name="RH_HFE">
-          <command_interface name="effort"/>
-          <state_interface name="position"/>
-          <state_interface name="velocity"/>
-          <param name="command_interface">position</param>
-      </joint>
-      <joint name="RH_KFE">
-          <command_interface name="effort"/>
-          <state_interface name="position"/>
-          <state_interface name="velocity"/>
-          <param name="command_interface">position</param>
-      </joint>
-      <joint name="LH_HAA">
-          <command_interface name="effort"/>
-          <state_interface name="position"/>
-          <state_interface name="velocity"/>
-          <param name="command_interface">position</param>
-      </joint>
-      <joint name="LH_HFE">
-          <command_interface name="effort"/>
-          <state_interface name="position"/>
-          <state_interface name="velocity"/>
-          <param name="command_interface">position</param>
-      </joint>
-      <joint name="LH_KFE">
-          <command_interface name="effort"/>
-          <state_interface name="position"/>
-          <state_interface name="velocity"/>
-      </joint>
-      <!-- Ankles mimic KFE joints -->
-      <joint name="LF_ankle">
-          <state_interface name="position"/>
-          <state_interface name="velocity"/>
-      </joint>
-      <joint name="LH_ankle">
-          <state_interface name="position"/>
-          <state_interface name="velocity"/>
-      </joint>
-      <joint name="RH_ankle">
-          <state_interface name="position"/>
-          <state_interface name="velocity"/>
-      </joint>
-      <!-- Control Rods mimic KFE joints -->
-      <joint name="fr_control_rod">
-          <state_interface name="position"/>
-          <state_interface name="velocity"/>
-      </joint>
-      <joint name="fl_control_rod">
-          <state_interface name="position"/>
-          <state_interface name="velocity"/>
-      </joint>
-      <joint name="br_control_rod">
-          <state_interface name="position"/>
-          <state_interface name="velocity"/>
-      </joint>
-      <joint name="bl_control_rod">
-          <state_interface name="position"/>
-          <state_interface name="velocity"/>
-      </joint>
-  </ros2_control>
+  <hardware>
+    <plugin>gz_ros2_control/GazeboSimSystem</plugin>
+    <param name="command_interface">position</param>
+    <param name="command_interface">effort</param>
+    <param name="update_rate">1000</param>
+  </hardware>
+  <!-- 12 Actuated Joints -->
+  <joint name="RF_HAA">
+    <command_interface name="effort"/>
+    <command_interface name="position"/>
+    <state_interface name="position"/>
+    <state_interface name="velocity"/>
+  </joint>
+  <joint name="RF_HFE">
+    <command_interface name="effort"/>
+    <command_interface name="position"/>
+    <state_interface name="position"/>
+    <state_interface name="velocity"/>
+  </joint>
+  <joint name="RF_KFE">
+    <command_interface name="effort"/>
+    <command_interface name="position"/>
+    <state_interface name="position"/>
+    <state_interface name="velocity"/>
+  </joint>
+  <joint name="LF_HAA">
+    <command_interface name="effort"/>
+    <command_interface name="position"/>
+    <state_interface name="position"/>
+    <state_interface name="velocity"/>
+  </joint>
+  <joint name="LF_HFE">
+    <command_interface name="effort"/>
+    <command_interface name="position"/>
+    <state_interface name="position"/>
+    <state_interface name="velocity"/>
+  </joint>
+  <joint name="LF_KFE">
+    <command_interface name="effort"/>
+    <command_interface name="position"/>
+    <state_interface name="position"/>
+    <state_interface name="velocity"/>
+  </joint>
+  <joint name="RH_HAA">
+    <command_interface name="effort"/>
+    <command_interface name="position"/>
+    <state_interface name="position"/>
+    <state_interface name="velocity"/>
+  </joint>
+  <joint name="RH_HFE">
+    <command_interface name="effort"/>
+    <command_interface name="position"/>
+    <state_interface name="position"/>
+    <state_interface name="velocity"/>
+  </joint>
+  <joint name="RH_KFE">
+    <command_interface name="effort"/>
+    <command_interface name="position"/>
+    <state_interface name="position"/>
+    <state_interface name="velocity"/>
+  </joint>
+  <joint name="LH_HAA">
+    <command_interface name="effort"/>
+    <command_interface name="position"/>
+    <state_interface name="position"/>
+    <state_interface name="velocity"/>
+  </joint>
+  <joint name="LH_HFE">
+    <command_interface name="effort"/>
+    <command_interface name="position"/>
+    <state_interface name="position"/>
+    <state_interface name="velocity"/>
+  </joint>
+  <joint name="LH_KFE">
+    <command_interface name="effort"/>
+    <command_interface name="position"/>
+    <state_interface name="position"/>
+    <state_interface name="velocity"/>
+  </joint>
+  <!-- Mimic joints (only state interfaces) -->
+  <joint name="LF_ankle">
+    <state_interface name="position"/>
+    <state_interface name="velocity"/>
+  </joint>
+  <joint name="LH_ankle">
+    <state_interface name="position"/>
+    <state_interface name="velocity"/>
+  </joint>
+  <joint name="RH_ankle">
+    <state_interface name="position"/>
+    <state_interface name="velocity"/>
+  </joint>
+  <joint name="fr_control_rod">
+    <state_interface name="position"/>
+    <state_interface name="velocity"/>
+  </joint>
+  <joint name="fl_control_rod">
+    <state_interface name="position"/>
+    <state_interface name="velocity"/>
+  </joint>
+  <joint name="br_control_rod">
+    <state_interface name="position"/>
+    <state_interface name="velocity"/>
+  </joint>
+  <joint name="bl_control_rod">
+    <state_interface name="position"/>
+    <state_interface name="velocity"/>
+  </joint>
+</ros2_control>
   <joint type="fixed" name="camera_joint">
     <origin xyz="0.225 0 0.075" rpy="0 0 0"/>
@@ -1318,5 +1339,4 @@
   <link name="camera_link_optical">
   </link>
-  <!-- STEP 8 - IMU -->
   <joint name="imu_joint" type="fixed">
     <origin xyz="0 0 0" rpy="0 0 0" />
